File: hardware/pcb/HitteStress2023_pcb/HitteStress2023_pcb.kicad_pcb (KiCad board)
At the start: 2 copper layers, 152.4 x 63.5 mm, 8 parts, among them J1 Conn_01x02_Socket, J2 Conn_01x02_Socket, J3 SMA_conector_female, U1 MINIDCDCBOOST5V, U2 TTGO T-Beam T22 V1.1

Commit message: Update design with IoT-Apeldoorn logo
Parts:
- added G***: LOGO, my-KiCad-library:IOT-Apeldoorn_Logo_22x9_6mm_silk, F.Cu at (146.1, 85.1)

Commit message: Updated PCB
Parts:
- added G***: LOGO_LogoRFSee_28x5-6mm, my-KiCad-library:LOGO_LogoRFSee_28x5-6mm, F.Cu at (140.7, 55.7)
Routing:
- net /GND: track 259.9 -> 260.5 mm, vias 71 -> 118
- net /SCL: track 115.1 -> 115.6 mm
Other:
- board text added: "ANT"
- board text added: "Hittestress 2023"
- board text added: "info@iot-apeldoorn.nl"
